Commit message: Make transmissions ros_control compatible
The transmission style changed for ros_control, the transmissions
need a type element a joint element with a hardware interface and
an actuator.

File: pr2_description/urdf/base_v0/base.transmission.xacro (robot description, xacro)
@@ -6,16 +6,24 @@
   <!--  Caster wheel transmission   -->
   <xacro:macro name="pr2_wheel_transmission_v0" params="suffix parent reflect">
-    <transmission type="pr2_mechanism_model/SimpleTransmission" name="${parent}_${suffix}_wheel_trans">
-      <actuator name="${parent}_${suffix}_wheel_motor" />
-      <joint name="${parent}_${suffix}_wheel_joint" />
-      <mechanicalReduction>${reflect * 624/35 * 80/18}</mechanicalReduction>
+    <transmission  name="${parent}_${suffix}_wheel_trans">
+      <type>pr2_mechanism_model/SimpleTransmission</type>
+      <actuator name="${parent}_${suffix}_wheel_motor">
+        <mechanicalReduction>${reflect * 624/35 * 80/18}</mechanicalReduction>
+      </actuator>
+      <joint name="${parent}_${suffix}_wheel_joint">
+        <hardwareInterface>EffortJointInterface</hardwareInterface>
+      </joint>
     </transmission>
   </xacro:macro>
   <!-- Hub transmission only -->
   <xacro:macro name="pr2_caster_transmission_v0" params="suffix">
-    <transmission type="pr2_mechanism_model/SimpleTransmission" name="${suffix}_rotation_trans">
-      <actuator name="${suffix}_rotation_motor" />
-      <joint name="${suffix}_rotation_joint" />
-      <mechanicalReduction>${-1 * 624/35 * 80/18}</mechanicalReduction>
+    <transmission name="${suffix}_rotation_trans">
+      <type>pr2_mechanism_model/SimpleTransmission</type>
+      <actuator name="${suffix}_rotation_motor">
+        <mechanicalReduction>${-1 * 624/35 * 80/18}</mechanicalReduction>
+      </actuator>
+      <joint name="${suffix}_rotation_joint">
+        <hardwareInterface>EffortJointInterface</hardwareInterface>
+      </joint>
     </transmission>
   </xacro:macro>

File: pr2_description/urdf/forearm_v0/forearm.transmission.xacro (robot description, xacro)
@@ -7,4 +7,11 @@
     <!-- Wrist flex , Wrist roll -->
     <transmission type="pr2_mechanism_model/WristTransmission" name="${side}_wrist_trans">
+      <type>pr2_mechanism_model/WristTransmission</type>
+      <joint name="${side}_wrist_r_joint">
+        <hardwareInterface>EffortJointInterface</hardwareInterface>
+      </joint>
+      <actuator name="${side}_wrist_r_motor">
+        <mechanicalReduction>1.0</mechanicalReduction>
+      </actuator>
       <rightActuator name="${side}_wrist_r_motor" mechanicalReduction="${624/35*54/16}"/>
       <leftActuator name="${side}_wrist_l_motor"  mechanicalReduction="${624/35*54/16}"/>

File: pr2_description/urdf/gripper_v0/gripper.transmission.xacro (robot description, xacro)
@@ -15,6 +15,12 @@
     <!-- Please refer to mechanism_model/src/pr2_gripper_transmission.cpp for implementation.-->
     <!-- gazebo_mimic_pid is for sim only.                                                   -->
-    <transmission type="pr2_mechanism_model/PR2GripperTransmission" name="${side}_gripper_trans" >
-      <actuator       name="${side}_gripper_motor" />
+    <transmission name="${side}_gripper_trans" >
+      <type>pr2_mechanism_model/PR2GripperTransmission</type>
+      <joint name="${side}_gripper_joint">
+        <hardwareInterface>EffortJointInterface</hardwareInterface>
+      </joint>
+      <actuator       name="${side}_gripper_motor">
+        <mechanicalReduction>1.0</mechanicalReduction>
+      </actuator>
       <gap_joint      name="${side}_gripper_joint"
                       mechanical_reduction="1.0"

File: pr2_description/urdf/head_v0/head.transmission.xacro (robot description, xacro)
@@ -5,15 +5,23 @@
        xmlns:xacro="http://ros.org/wiki/xacro">
   <xacro:macro name="pr2_head_pan_transmission_v0" params="name">
-    <transmission type="pr2_mechanism_model/SimpleTransmission" name="${name}_trans">
-      <actuator name="${name}_motor" />
-      <joint name="${name}_joint" />
-      <mechanicalReduction>6.0</mechanicalReduction>
+    <transmission name="${name}_trans">
+      <type>pr2_mechanism_model/SimpleTransmission</type>
+      <actuator name="${name}_motor">
+        <mechanicalReduction>6.0</mechanicalReduction>
+      </actuator>
+      <joint name="${name}_joint">
+        <hardwareInterface>EffortJointInterface</hardwareInterface>
+      </joint>
     </transmission>
   </xacro:macro>
   <xacro:macro name="pr2_head_tilt_transmission_v0" params="name">
-    <transmission type="pr2_mechanism_model/SimpleTransmission" name="${name}_trans">
-      <actuator name="${name}_motor" />
-      <joint name="${name}_joint" />
-      <mechanicalReduction>6.0</mechanicalReduction>
+    <transmission name="${name}_trans">
+      <type>pr2_mechanism_model/SimpleTransmission</type>
+      <actuator name="${name}_motor">
+        <mechanicalReduction>6.0</mechanicalReduction>
+      </actuator>
+      <joint name="${name}_joint">
+        <hardwareInterface>EffortJointInterface</hardwareInterface>
+      </joint>
     </transmission>
   </xacro:macro>

File: pr2_description/urdf/shoulder_v0/shoulder.transmission.xacro (robot description, xacro)
@@ -6,15 +6,23 @@
   <xacro:macro name="pr2_shoulder_transmission_v0" params="side">
     <!-- Shoulder pan -->
-    <transmission type="pr2_mechanism_model/SimpleTransmission" name="${side}_shoulder_pan_trans">
-      <joint name="${side}_shoulder_pan_joint"/>
-      <actuator name="${side}_shoulder_pan_motor"/>
-      <mechanicalReduction>${13/3 * 250.532/17.19 / cal_r_shoulder_pan_gearing}</mechanicalReduction>
+    <transmission name="${side}_shoulder_pan_trans">
+      <type>pr2_mechanism_model/SimpleTransmission</type>
+      <joint name="${side}_shoulder_pan_joint">
+        <hardwareInterface>EffortJointInterface</hardwareInterface>
+      </joint>
+      <actuator name="${side}_shoulder_pan_motor">
+        <mechanicalReduction>${13/3 * 250.532/17.19 / cal_r_shoulder_pan_gearing}</mechanicalReduction>
+      </actuator>
       <compensator k_belt="4000.0" mass_motor="0.05" kd_motor="15.0" lambda_motor="40.0" lambda_joint="40.0" lambda_combined="0.0"/>
     </transmission>
     <!-- Shoulder lift -->
-    <transmission type="pr2_mechanism_model/SimpleTransmission" name="${side}_shoulder_lift_trans">
-      <joint name="${side}_shoulder_lift_joint"/>
-      <actuator name="${side}_shoulder_lift_motor"/>
-      <mechanicalReduction>${13/3 * 245.532/17.19 / cal_r_shoulder_lift_gearing}</mechanicalReduction>
+    <transmission name="${side}_shoulder_lift_trans">
+      <type>pr2_mechanism_model/SimpleTransmission</type>
+      <joint name="${side}_shoulder_lift_joint">
+        <hardwareInterface>EffortJointInterface</hardwareInterface>
+      </joint>
+      <actuator name="${side}_shoulder_lift_motor">
+        <mechanicalReduction>${13/3 * 245.532/17.19 / cal_r_shoulder_lift_gearing}</mechanicalReduction>
+      </actuator>
       <compensator k_belt="4000.0" mass_motor="0.05" kd_motor="10.0" lambda_motor="60.0" lambda_joint="60.0" lambda_combined="0.0"/>
     </transmission>
@@ -22,8 +30,12 @@
   <xacro:macro name="pr2_upper_arm_roll_transmission_v0" params="side" >
     <!-- Upperarm roll: internal fixed attchment point for upper arm -->
-    <transmission type="pr2_mechanism_model/SimpleTransmission" name="${side}_upper_arm_roll_trans">
-      <actuator name="${side}_upper_arm_roll_motor" />
-      <joint name="${side}_upper_arm_roll_joint" />
-      <mechanicalReduction>${13/3 * 129.53/17.19 / cal_r_upper_arm_roll_gearing}</mechanicalReduction>
+    <transmission name="${side}_upper_arm_roll_trans">
+      <type>pr2_mechanism_model/SimpleTransmission</type>
+      <actuator name="${side}_upper_arm_roll_motor">
+        <mechanicalReduction>${13/3 * 129.53/17.19 / cal_r_upper_arm_roll_gearing}</mechanicalReduction>
+      </actuator>
+      <joint name="${side}_upper_arm_roll_joint">
+        <hardwareInterface>EffortJointInterface</hardwareInterface>
+      </joint>
     </transmission>
   </xacro:macro>

File: pr2_description/urdf/tilting_laser_v0/tilting_laser.transmission.xacro (robot description, xacro)
@@ -5,8 +5,12 @@
        xmlns:xacro="http://ros.org/wiki/xacro">
   <xacro:macro name="pr2_tilting_laser_transmission_v0" params="name">
-    <transmission type="pr2_mechanism_model/SimpleTransmission" name="${name}_mount_trans">
-      <actuator name="${name}_mount_motor" />
-      <joint name="${name}_mount_joint" />
-      <mechanicalReduction>-6.05</mechanicalReduction>
+    <transmission name="${name}_mount_trans">
+      <type>pr2_mechanism_model/SimpleTransmission</type>
+      <actuator name="${name}_mount_motor">
+        <mechanicalReduction>-6.05</mechanicalReduction>
+      </actuator>
+      <joint name="${name}_mount_joint">
+        <hardwareInterface>EffortJointInterface</hardwareInterface>
+      </joint>
     </transmission>
   </xacro:macro>

File: pr2_description/urdf/torso_v0/torso.transmission.xacro (robot description, xacro)
@@ -5,8 +5,12 @@
        xmlns:xacro="http://ros.org/wiki/xacro">
   <xacro:macro name="pr2_torso_transmission_v0" params="name">
-    <transmission type="pr2_mechanism_model/SimpleTransmission" name="${name}_trans">
-      <actuator name="${name}_motor" />
-      <joint name="${name}_joint" />
-      <mechanicalReduction>-47641.53</mechanicalReduction>
+    <transmission name="${name}_trans">
+      <type>pr2_mechanism_model/SimpleTransmission</type>
+      <actuator name="${name}_motor">
+        <mechanicalReduction>-47641.53</mechanicalReduction>
+      </actuator>
+      <joint name="${name}_joint">
+        <hardwareInterface>EffortJointInterface</hardwareInterface>
+      </joint>
       <simulated_actuated_joint name="${name}_motor_screw_joint"
                                 simulated_reduction="3141.6" />

File: pr2_description/urdf/upper_arm_v0/upper_arm.transmission.xacro (robot description, xacro)
@@ -7,16 +7,24 @@
   <xacro:macro name="pr2_elbow_flex_transmission_v0" params="side">
     <!-- Elbow flex -->
-    <transmission type="pr2_mechanism_model/SimpleTransmission" name="${side}_elbow_flex_trans">
-      <actuator name="${side}_elbow_flex_motor" />
-      <joint name="${side}_elbow_flex_joint" />
-      <mechanicalReduction>${-13/3 * 127.532/15.28}</mechanicalReduction>
+    <transmission name="${side}_elbow_flex_trans">
+      <type>pr2_mechanism_model/SimpleTransmission</type>
+      <actuator name="${side}_elbow_flex_motor">
+        <mechanicalReduction>${-13/3 * 127.532/15.28}</mechanicalReduction>
+      </actuator>
+      <joint name="${side}_elbow_flex_joint">
+        <hardwareInterface>EffortJointInterface</hardwareInterface>
+      </joint>
     </transmission>
   </xacro:macro>
   <!-- Forearm roll -->
   <xacro:macro name="pr2_forearm_roll_transmission_v0" params="side" >
-    <transmission type="pr2_mechanism_model/SimpleTransmission" name="${side}_forearm_roll_trans">
-      <actuator name="${side}_forearm_roll_motor" />
-      <joint name="${side}_forearm_roll_joint" />
-      <mechanicalReduction>${-576/25 * 55/14}</mechanicalReduction>
+    <transmission name="${side}_forearm_roll_trans">
+      <type>pr2_mechanism_model/SimpleTransmission</type>
+      <actuator name="${side}_forearm_roll_motor">
+        <mechanicalReduction>${-576/25 * 55/14}</mechanicalReduction>
+      </actuator>
+      <joint name="${side}_forearm_roll_joint">
+        <hardwareInterface>EffortJointInterface</hardwareInterface>
+      </joint>
     </transmission>
   </xacro:macro>

Commit message: Make transmissions ros_control compatible
The transmission style changed for ros_control, the transmissions
need a type element a joint element with a hardware interface and
an actuator.

File: pr2_description/urdf/base_v0/base.transmission.xacro (robot description, xacro)
@@ -3,16 +3,24 @@
   <!--  Caster wheel transmission   -->
   <xacro:macro name="pr2_wheel_transmission_v0" params="suffix parent reflect">
-    <transmission type="pr2_mechanism_model/SimpleTransmission" name="${parent}_${suffix}_wheel_trans">
-      <actuator name="${parent}_${suffix}_wheel_motor" />
-      <joint name="${parent}_${suffix}_wheel_joint" />
-      <mechanicalReduction>${reflect * 624/35 * 80/18}</mechanicalReduction>
+    <transmission  name="${parent}_${suffix}_wheel_trans">
+      <type>pr2_mechanism_model/SimpleTransmission</type>
+      <actuator name="${parent}_${suffix}_wheel_motor">
+        <mechanicalReduction>${reflect * 624/35 * 80/18}</mechanicalReduction>
+      </actuator>
+      <joint name="${parent}_${suffix}_wheel_joint">
+        <hardwareInterface>EffortJointInterface</hardwareInterface>
+      </joint>
     </transmission>
   </xacro:macro>
   <!-- Hub transmission only -->
   <xacro:macro name="pr2_caster_transmission_v0" params="suffix">
-    <transmission type="pr2_mechanism_model/SimpleTransmission" name="${suffix}_rotation_trans">
-      <actuator name="${suffix}_rotation_motor" />
-      <joint name="${suffix}_rotation_joint" />
-      <mechanicalReduction>${-1 * 624/35 * 80/18}</mechanicalReduction>
+    <transmission name="${suffix}_rotation_trans">
+      <type>pr2_mechanism_model/SimpleTransmission</type>
+      <actuator name="${suffix}_rotation_motor">
+        <mechanicalReduction>${-1 * 624/35 * 80/18}</mechanicalReduction>
+      </actuator>
+      <joint name="${suffix}_rotation_joint">
+        <hardwareInterface>EffortJointInterface</hardwareInterface>
+      </joint>
     </transmission>
   </xacro:macro>

File: pr2_description/urdf/forearm_v0/forearm.transmission.xacro (robot description, xacro)
@@ -4,4 +4,11 @@
     <!-- Wrist flex , Wrist roll -->
     <transmission type="pr2_mechanism_model/WristTransmission" name="${side}_wrist_trans">
+      <type>pr2_mechanism_model/WristTransmission</type>
+      <joint name="${side}_wrist_r_joint">
+        <hardwareInterface>EffortJointInterface</hardwareInterface>
+      </joint>
+      <actuator name="${side}_wrist_r_motor">
+        <mechanicalReduction>1.0</mechanicalReduction>
+      </actuator>
       <rightActuator name="${side}_wrist_r_motor" mechanicalReduction="${624/35*54/16}"/>
       <leftActuator name="${side}_wrist_l_motor"  mechanicalReduction="${624/35*54/16}"/>

File: pr2_description/urdf/gripper_v0/gripper.transmission.xacro (robot description, xacro)
@@ -11,6 +11,12 @@
     <!-- Please refer to mechanism_model/src/pr2_gripper_transmission.cpp for implementation.-->
     <!-- gazebo_mimic_pid is for sim only.                                                   -->
-    <transmission type="pr2_mechanism_model/PR2GripperTransmission" name="${side}_gripper_trans" >
-      <actuator       name="${side}_gripper_motor" />
+    <transmission name="${side}_gripper_trans" >
+      <type>pr2_mechanism_model/PR2GripperTransmission</type>
+      <joint name="${side}_gripper_joint">
+        <hardwareInterface>EffortJointInterface</hardwareInterface>
+      </joint>
+      <actuator       name="${side}_gripper_motor">
+        <mechanicalReduction>1.0</mechanicalReduction>
+      </actuator>
       <gap_joint      name="${side}_gripper_joint"
                       mechanical_reduction="1.0"

File: pr2_description/urdf/head_v0/head.transmission.xacro (robot description, xacro)
@@ -2,15 +2,23 @@
 <robot xmlns:xacro="http://www.ros.org/wiki/xacro">
   <xacro:macro name="pr2_head_pan_transmission_v0" params="name">
-    <transmission type="pr2_mechanism_model/SimpleTransmission" name="${name}_trans">
-      <actuator name="${name}_motor" />
-      <joint name="${name}_joint" />
-      <mechanicalReduction>6.0</mechanicalReduction>
+    <transmission name="${name}_trans">
+      <type>pr2_mechanism_model/SimpleTransmission</type>
+      <actuator name="${name}_motor">
+        <mechanicalReduction>6.0</mechanicalReduction>
+      </actuator>
+      <joint name="${name}_joint">
+        <hardwareInterface>EffortJointInterface</hardwareInterface>
+      </joint>
     </transmission>
   </xacro:macro>
   <xacro:macro name="pr2_head_tilt_transmission_v0" params="name">
-    <transmission type="pr2_mechanism_model/SimpleTransmission" name="${name}_trans">
-      <actuator name="${name}_motor" />
-      <joint name="${name}_joint" />
-      <mechanicalReduction>6.0</mechanicalReduction>
+    <transmission name="${name}_trans">
+      <type>pr2_mechanism_model/SimpleTransmission</type>
+      <actuator name="${name}_motor">
+        <mechanicalReduction>6.0</mechanicalReduction>
+      </actuator>
+      <joint name="${name}_joint">
+        <hardwareInterface>EffortJointInterface</hardwareInterface>
+      </joint>
     </transmission>
   </xacro:macro>

File: pr2_description/urdf/shoulder_v0/shoulder.transmission.xacro (robot description, xacro)
@@ -3,15 +3,23 @@
   <xacro:macro name="pr2_shoulder_transmission_v0" params="side">
     <!-- Shoulder pan -->
-    <transmission type="pr2_mechanism_model/SimpleTransmission" name="${side}_shoulder_pan_trans">
-      <joint name="${side}_shoulder_pan_joint"/>
-      <actuator name="${side}_shoulder_pan_motor"/>
-      <mechanicalReduction>${13/3 * 250.532/17.19 / cal_r_shoulder_pan_gearing}</mechanicalReduction>
+    <transmission name="${side}_shoulder_pan_trans">
+      <type>pr2_mechanism_model/SimpleTransmission</type>
+      <joint name="${side}_shoulder_pan_joint">
+        <hardwareInterface>EffortJointInterface</hardwareInterface>
+      </joint>
+      <actuator name="${side}_shoulder_pan_motor">
+        <mechanicalReduction>${13/3 * 250.532/17.19 / cal_r_shoulder_pan_gearing}</mechanicalReduction>
+      </actuator>
       <compensator k_belt="4000.0" mass_motor="0.05" kd_motor="15.0" lambda_motor="40.0" lambda_joint="40.0" lambda_combined="0.0"/>
     </transmission>
     <!-- Shoulder lift -->
-    <transmission type="pr2_mechanism_model/SimpleTransmission" name="${side}_shoulder_lift_trans">
-      <joint name="${side}_shoulder_lift_joint"/>
-      <actuator name="${side}_shoulder_lift_motor"/>
-      <mechanicalReduction>${13/3 * 245.532/17.19 / cal_r_shoulder_lift_gearing}</mechanicalReduction>
+    <transmission name="${side}_shoulder_lift_trans">
+      <type>pr2_mechanism_model/SimpleTransmission</type>
+      <joint name="${side}_shoulder_lift_joint">
+        <hardwareInterface>EffortJointInterface</hardwareInterface>
+      </joint>
+      <actuator name="${side}_shoulder_lift_motor">
+        <mechanicalReduction>${13/3 * 245.532/17.19 / cal_r_shoulder_lift_gearing}</mechanicalReduction>
+      </actuator>
       <compensator k_belt="4000.0" mass_motor="0.05" kd_motor="10.0" lambda_motor="60.0" lambda_joint="60.0" lambda_combined="0.0"/>
     </transmission>
@@ -19,8 +27,12 @@
   <xacro:macro name="pr2_upper_arm_roll_transmission_v0" params="side" >
     <!-- Upperarm roll: internal fixed attchment point for upper arm -->
-    <transmission type="pr2_mechanism_model/SimpleTransmission" name="${side}_upper_arm_roll_trans">
-      <actuator name="${side}_upper_arm_roll_motor" />
-      <joint name="${side}_upper_arm_roll_joint" />
-      <mechanicalReduction>${13/3 * 129.53/17.19 / cal_r_upper_arm_roll_gearing}</mechanicalReduction>
+    <transmission name="${side}_upper_arm_roll_trans">
+      <type>pr2_mechanism_model/SimpleTransmission</type>
+      <actuator name="${side}_upper_arm_roll_motor">
+        <mechanicalReduction>${13/3 * 129.53/17.19 / cal_r_upper_arm_roll_gearing}</mechanicalReduction>
+      </actuator>
+      <joint name="${side}_upper_arm_roll_joint">
+        <hardwareInterface>EffortJointInterface</hardwareInterface>
+      </joint>
     </transmission>
   </xacro:macro>

File: pr2_description/urdf/tilting_laser_v0/tilting_laser.transmission.xacro (robot description, xacro)
@@ -2,8 +2,12 @@
 <robot xmlns:xacro="http://www.ros.org/wiki/xacro">
   <xacro:macro name="pr2_tilting_laser_transmission_v0" params="name">
-    <transmission type="pr2_mechanism_model/SimpleTransmission" name="${name}_mount_trans">
-      <actuator name="${name}_mount_motor" />
-      <joint name="${name}_mount_joint" />
-      <mechanicalReduction>-6.05</mechanicalReduction>
+    <transmission name="${name}_mount_trans">
+      <type>pr2_mechanism_model/SimpleTransmission</type>
+      <actuator name="${name}_mount_motor">
+        <mechanicalReduction>-6.05</mechanicalReduction>
+      </actuator>
+      <joint name="${name}_mount_joint">
+        <hardwareInterface>EffortJointInterface</hardwareInterface>
+      </joint>
     </transmission>
   </xacro:macro>

File: pr2_description/urdf/torso_v0/torso.transmission.xacro (robot description, xacro)
@@ -2,8 +2,12 @@
 <robot xmlns:xacro="http://www.ros.org/wiki/xacro">
   <xacro:macro name="pr2_torso_transmission_v0" params="name">
-    <transmission type="pr2_mechanism_model/SimpleTransmission" name="${name}_trans">
-      <actuator name="${name}_motor" />
-      <joint name="${name}_joint" />
-      <mechanicalReduction>-47641.53</mechanicalReduction>
+    <transmission name="${name}_trans">
+      <type>pr2_mechanism_model/SimpleTransmission</type>
+      <actuator name="${name}_motor">
+        <mechanicalReduction>-47641.53</mechanicalReduction>
+      </actuator>
+      <joint name="${name}_joint">
+        <hardwareInterface>EffortJointInterface</hardwareInterface>
+      </joint>
       <simulated_actuated_joint name="${name}_motor_screw_joint"
                                 simulated_reduction="3141.6" />

File: pr2_description/urdf/upper_arm_v0/upper_arm.transmission.xacro (robot description, xacro)
@@ -4,16 +4,24 @@
   <xacro:macro name="pr2_elbow_flex_transmission_v0" params="side">
     <!-- Elbow flex -->
-    <transmission type="pr2_mechanism_model/SimpleTransmission" name="${side}_elbow_flex_trans">
-      <actuator name="${side}_elbow_flex_motor" />
-      <joint name="${side}_elbow_flex_joint" />
-      <mechanicalReduction>${-13/3 * 127.532/15.28}</mechanicalReduction>
+    <transmission name="${side}_elbow_flex_trans">
+      <type>pr2_mechanism_model/SimpleTransmission</type>
+      <actuator name="${side}_elbow_flex_motor">
+        <mechanicalReduction>${-13/3 * 127.532/15.28}</mechanicalReduction>
+      </actuator>
+      <joint name="${side}_elbow_flex_joint">
+        <hardwareInterface>EffortJointInterface</hardwareInterface>
+      </joint>
     </transmission>
   </xacro:macro>
   <!-- Forearm roll -->
   <xacro:macro name="pr2_forearm_roll_transmission_v0" params="side" >
-    <transmission type="pr2_mechanism_model/SimpleTransmission" name="${side}_forearm_roll_trans">
-      <actuator name="${side}_forearm_roll_motor" />
-      <joint name="${side}_forearm_roll_joint" />
-      <mechanicalReduction>${-576/25 * 55/14}</mechanicalReduction>
+    <transmission name="${side}_forearm_roll_trans">
+      <type>pr2_mechanism_model/SimpleTransmission</type>
+      <actuator name="${side}_forearm_roll_motor">
+        <mechanicalReduction>${-576/25 * 55/14}</mechanicalReduction>
+      </actuator>
+      <joint name="${side}_forearm_roll_joint">
+        <hardwareInterface>EffortJointInterface</hardwareInterface>
+      </joint>
     </transmission>
   </xacro:macro>
