Commit message: use absolute calibration values
the calibration_estimation created calibration offsets to the last calibration
we extended the script, now it creates a yaml file with the new absolut valus.
These are used in the xacro files now

File: pr2_description/urdf/base_v0/base.urdf.xacro (robot description, xacro)
@@ -80,5 +80,5 @@
       <safety_controller  k_velocity="10" />
       <xacro:if value="$(arg calibrated)">
-        <calibration falling="${ref_position + calibration_data['transforms'][suffix+'_rotation_joint'][5]}" />
+        <calibration falling="${calibration_data['calibration'][suffix+'_rotation_joint']}" />
       </xacro:if>
       <xacro:unless value="$(arg calibrated)">

File: pr2_description/urdf/head_v0/head.urdf.xacro (robot description, xacro)
@@ -13,5 +13,5 @@
       <safety_controller k_velocity="1.5" soft_lower_limit="${-3.007+0.15}" soft_upper_limit="${3.007-0.15}" k_position="100" />
       <xacro:if value="$(arg calibrated)">
-        <calibration falling="${0.0 + calibration_data['transforms'][name+'_joint'][5]}" />
+        <calibration falling="${calibration_data['calibration'][name+'_joint']}" />
       </xacro:if>
       <xacro:unless value="$(arg calibrated)">
@@ -52,5 +52,5 @@
       <safety_controller k_velocity="3.0" soft_lower_limit="${-0.4712 + 0.1}" soft_upper_limit="${1.39626 - 0.1}" k_position="100" />
       <xacro:if value="$(arg calibrated)">
-        <calibration falling="${0.0+cal_head_tilt_flag + calibration_data['transforms'][name+'_joint'][4]}" />
+        <calibration falling="${calibration_data['calibration'][name+'_joint']}" />
       </xacro:if>
       <xacro:unless value="$(arg calibrated)">

File: pr2_description/urdf/sensors/double_stereo_camera.urdf.xacro (robot description, xacro)
@@ -40,8 +40,20 @@
     <!-- 15mm offset from center needs check with CAD -->
     <xacro:stereo_camera_v0 parent="${name}_link" name="wide_stereo" focal_length="320.000105" hfov="90" image_format="BAYER_BGGR8" image_width="640" image_height="480" >
-      <origin xyz="0.045 ${0.045-0.015} 0.0501" rpy="0.0   0.0   0.0" />
+      <xacro:if value="$(arg calibrated)">
+        <origin xyz="${calibration_data['transforms']['xyz']['wide_stereo_frame_joint'][0]} ${calibration_data['transforms']['xyz']['wide_stereo_frame_joint'][1]} ${calibration_data['transforms']['xyz']['wide_stereo_frame_joint'][2]}"
+                rpy="${calibration_data['transforms']['rpy']['wide_stereo_frame_joint'][0]} ${calibration_data['transforms']['rpy']['wide_stereo_frame_joint'][1]} ${calibration_data['transforms']['rpy']['wide_stereo_frame_joint'][2]}" />
+      </xacro:if>
+      <xacro:unless value="$(arg calibrated)">
+        <origin xyz="0.045 ${0.045-0.015} 0.0501" rpy="0.0   0.0   0.0" />
+      </xacro:unless>
     </xacro:stereo_camera_v0>
     <xacro:stereo_camera_v0 parent="${name}_link" name="narrow_stereo" focal_length="772.548518" hfov="45" image_format="L8" image_width="640" image_height="480" >
-      <origin xyz="0.045 ${0.045+0.015} 0.0501" rpy="0.0   0.0   0.0" />
+      <xacro:if value="$(arg calibrated)">
+        <origin xyz="${calibration_data['transforms']['xyz']['narrow_stereo_frame_joint'][0]} ${calibration_data['transforms']['xyz']['narrow_stereo_frame_joint'][1]} ${calibration_data['transforms']['xyz']['narrow_stereo_frame_joint'][2]}"
+                rpy="${calibration_data['transforms']['rpy']['narrow_stereo_frame_joint'][0]} ${calibration_data['transforms']['rpy']['narrow_stereo_frame_joint'][1]} ${calibration_data['transforms']['rpy']['narrow_stereo_frame_joint'][2]}" />
+      </xacro:if>
+      <xacro:unless value="$(arg calibrated)">
+        <origin xyz="0.045 ${0.045+0.015} 0.0501" rpy="0.0   0.0   0.0" />
+      </xacro:unless>
     </xacro:stereo_camera_v0>
     <!-- extensions -->

File: pr2_description/urdf/shoulder_v0/shoulder.urdf.xacro (robot description, xacro)
@@ -28,5 +28,5 @@
       <!-- joint angle when the rising or the falling flag is activated on PR2 -->
       <xacro:if value="$(arg calibrated)">
-        <calibration falling="${(reflect*M_PI/4)*cal_r_shoulder_pan_gearing+cal_r_shoulder_pan_flag + calibration_data['transforms'][side+'_shoulder_pan_joint'][5]}" />
+        <calibration falling="${calibration_data['calibration'][side+'_shoulder_pan_joint']}" />
       </xacro:if>
       <xacro:unless value="$(arg calibrated)">
@@ -65,5 +65,5 @@
                          soft_lower_limit="${-0.5236+0.17}" soft_upper_limit="${1.3963-0.10}" />
       <xacro:if value="$(arg calibrated)">
-        <calibration falling="${cal_r_shoulder_lift_flag + calibration_data['transforms'][side+'_shoulder_lift_joint'][4]}" />
+        <calibration falling="${calibration_data['calibration'][side+'_shoulder_lift_joint']}" />
       </xacro:if>
       <xacro:unless value="$(arg calibrated)">
@@ -115,5 +115,5 @@
       <safety_controller k_position="100" k_velocity="2" soft_lower_limit="${reflect*1.55-2.35+0.15}" soft_upper_limit="${reflect*1.55+2.35-0.15}" />
       <xacro:if value="$(arg calibrated)">
-        <calibration falling="${(reflect*M_PI/2)*cal_r_upper_arm_roll_gearing + cal_r_upper_arm_roll_flag + calibration_data['transforms'][side+'_upper_arm_roll_joint'][3]}" />
+        <calibration falling="${calibration_data['calibration'][side+'_upper_arm_roll_joint']}" />
       </xacro:if>
       <xacro:unless value="$(arg calibrated)">

File: pr2_description/urdf/tilting_laser_v0/tilting_laser.urdf.xacro (robot description, xacro)
@@ -13,5 +13,5 @@
       <safety_controller k_position="100" k_velocity="0.05" soft_lower_limit="${-0.7854+0.05}" soft_upper_limit="${1.48353-0.05}" />
       <xacro:if value="$(arg calibrated)">
-        <calibration falling="${laser_calib_ref + calibration_data['transforms'][name+'_mount_joint'][4]}" />
+        <calibration falling="${calibration_data['calibration'][name+'_mount_joint']}" />
       </xacro:if>
       <xacro:unless value="$(arg calibrated)">
@@ -46,5 +46,11 @@
     </link>
     <xacro:hokuyo_lx30_laser_v0 name="${name}" parent="${name}_mount" ros_topic="tilt_scan" update_rate="40" min_angle="-1.3962634" max_angle="1.3962634" >
-      <origin xyz="0 0 0.03" rpy="0 0 0" />
+      <xacro:if value="$(arg calibrated)">
+        <origin xyz="${calibration_data['transforms']['xyz'][name+'_joint'][0]} ${calibration_data['transforms']['xyz'][name+'_joint'][1]} ${calibration_data['transforms']['xyz'][name+'_joint'][2]}"
+                rpy="${calibration_data['transforms']['rpy'][name+'_joint'][0]} ${calibration_data['transforms']['rpy'][name+'_joint'][1]} ${calibration_data['transforms']['rpy'][name+'_joint'][2]}" />
+      </xacro:if>
+      <xacro:unless value="$(arg calibrated)">
+        <origin xyz="0 0 0.03" rpy="0 0 0" />
+      </xacro:unless>
     </xacro:hokuyo_lx30_laser_v0>
     <!-- extensions -->

File: pr2_description/urdf/torso_v0/torso.urdf.xacro (robot description, xacro)
@@ -13,5 +13,5 @@
       <safety_controller  k_velocity="2000000" soft_lower_limit="${0.0+0.0115}" soft_upper_limit="${0.33-0.005}" k_position="100" />
       <xacro:if value="$(arg calibrated)">
-        <calibration falling="${0.00475 + calibration_data['transforms'][name+'_joint'][5]}" />
+        <calibration falling="${calibration_data['calibration'][name+'_joint']}" />
       </xacro:if>
       <xacro:unless value="$(arg calibrated)">

File: pr2_description/urdf/upper_arm_v0/upper_arm.urdf.xacro (robot description, xacro)
@@ -78,5 +78,5 @@
       <safety_controller k_position="100" k_velocity="3" soft_lower_limit="${-2.3213+0.2}" soft_upper_limit="${0.00-0.15}" />
       <xacro:if value="$(arg calibrated)">
-        <calibration falling="${-1.1606 + cal_r_elbow_flex_flag + calibration_data['transforms'][side+'_elbow_flex_joint'][4]}" />
+        <calibration falling="${calibration_data['calibration'][side+'_elbow_flex_joint']}" />
       </xacro:if>
       <xacro:unless value="$(arg calibrated)">
@@ -121,5 +121,5 @@
       <safety_controller k_velocity="1" />
       <xacro:if value="$(arg calibrated)">
-        <calibration falling="${0.0 + cal_r_forearm_roll_flag + calibration_data['transforms'][side+'_forearm_roll_joint'][3]}" />
+        <calibration falling="${calibration_data['calibration'][side+'_forearm_roll_joint']}" />
       </xacro:if>
       <xacro:unless value="$(arg calibrated)">
