Commit message: Make transmissions ros_control compatible
The transmission style changed for ros_control, the transmissions
need a type element a joint element with a hardware interface and
an actuator.

File: pr2_description/urdf/gripper_v0/gripper.transmission.xacro (robot description, xacro)
@@ -11,6 +11,12 @@
     <!-- Please refer to mechanism_model/src/pr2_gripper_transmission.cpp for implementation.-->
     <!-- gazebo_mimic_pid is for sim only.                                                   -->
-    <transmission type="pr2_mechanism_model/PR2GripperTransmission" name="${side}_gripper_trans" >
-      <actuator       name="${side}_gripper_motor" />
+    <transmission name="${side}_gripper_trans" >
+      <type>pr2_mechanism_model/PR2GripperTransmission</type>
+      <joint name="${side}_gripper_joint">
+        <hardwareInterface>EffortJointInterface</hardwareInterface>
+      </joint>
+      <actuator       name="${side}_gripper_motor">
+        <mechanicalReduction>1.0</mechanicalReduction>
+      </actuator>
       <gap_joint      name="${side}_gripper_joint"
                       mechanical_reduction="1.0"
